Commit message: something doing

File: urdf/robot.urdf (robot description, URDF)
Before this commit: robot pick_and_drop_arm, 9 links, 8 joints
Joints:
- joint base_joint: origin xyz=0 0 0.1 -> xyz=0 0 0
- joint finger1_joint: axis 1 0 0 -> -1 0 0; limit lower=0 upper=0.8 effort=5 velocity=1.0 -> lower=-0.8 upper=0 effort=5 velocity=1.0; origin xyz=0.005756 -1.4504 -0.85021 -> xyz=0.005756 0.522025 1.59808
- joint finger2_joint: axis -1 0 0 -> 1 0 0; origin xyz=0.005756 -0.71318 -1.52533 -> xyz=0.005756 -0.477477 1.61468
- joint joint2: origin xyz=0 2.05731 2.08253 -> xyz=0 -0.007232 2.92735
- joint joint3: origin xyz=0 -2.041415 2.09397 -> xyz=0 0.002234 2.9244
- joint joint4: origin xyz=0 -2.104915 -0.30269 -> xyz=0 0.012929 2.12653
